File: analogFrontend.kicad_sch (KiCad schematic)
At the start: 0 parts

Commit message: Finished schematic of the FreqIn channels
Other:
- added sheet V Divider11 (analogInDivider.kicad_sch)
Changed lines of the file:
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@@
 (kicad_sch
-	(version 20250114)
+	(version 20260306)
 	(generator "eeschema")
-	(generator_version "9.0")
+	(generator_version "10.0")
 	(paper "A4")
 	(wire
@@
 	(wire
 		(pts
+			(xy 121.92 127) (xy 114.3 127)
+		)
+		(stroke
+			(width 0)
+			(type default)
+		)
+	)
+	(wire
+		(pts
 			(xy 114.3 58.42) (xy 121.92 58.42)
+		)
+		(stroke
+			(width 0)
+			(type default)
+		)
+	)
+	(wire
+		(pts
+			(xy 152.4 127) (xy 144.78 127)
 		)
 		(stroke
@@
 		)
 	)
+	(hierarchical_label "BAT+"
+		(shape input)
+		(at 152.4 127 0)
+		(effects
+			(font
+				(size 1.27 1.27)
+			)
+			(justify left)
+		)
+	)
 	(hierarchical_label "MCU_AN2"
 		(shape output)
@@
 		(shape output)
 		(at 114.3 96.52 180)
+		(effects
+			(font
+				(size 1.27 1.27)
+			)
+			(justify right)
+		)
+	)
+	(hierarchical_label "MCU_BAT+"
+		(shape output)
+		(at 114.3 127 180)
 		(effects
 			(font
@@
 		)
 		(fill
-			(color 0 0 0 0.0000)
+			(color 0 0 0 0)
 		)
 		(property "Sheetname" "V Divider"
 			(at 121.92 41.1984 0)
+			(show_name no)
+			(do_not_autoplace no)
 			(effects
 				(font
@@
 		(property "Sheetfile" "analogInDivider.kicad_sch"
 			(at 121.92 46.3046 0)
+			(hide yes)
+			(show_name no)
+			(do_not_autoplace no)
 			(effects
 				(font
@@
 				)
 				(justify left top)
-				(hide yes)
 			)
 		)
@@
 		)
 		(fill
-			(color 0 0 0 0.0000)
+			(color 0 0 0 0)
 		)
 		(property "Sheetname" "V Divider5"
 			(at 121.92 79.2984 0)
+			(show_name no)
+			(do_not_autoplace no)
 			(effects
 				(font
@@
 		(property "Sheetfile" "analogInDivider.kicad_sch"
 			(at 121.92 84.4046 0)
+			(hide yes)
+			(show_name no)
+			(do_not_autoplace no)
 			(effects
 				(font
@@
 				)
 				(justify left top)
-				(hide yes)
 			)
 		)
@@
 		)
 		(fill
-			(color 0 0 0 0.0000)
+			(color 0 0 0 0)
 		)
 		(property "Sheetname" "V Divider3"
 			(at 121.92 64.0584 0)
+			(show_name no)
+			(do_not_autoplace no)
 			(effects
 				(font
@@
 		(property "Sheetfile" "analogInDivider.kicad_sch"
 			(at 121.92 69.1646 0)
+			(hide yes)
+			(show_name no)
+			(do_not_autoplace no)
 			(effects
 				(font
@@
 				)
 				(justify left top)
-				(hide yes)
 			)
 		)
@@
 		)
 		(fill
-			(color 0 0 0 0.0000)
+			(color 0 0 0 0)
 		)
 		(property "Sheetname" "V Divider1"
 			(at 121.92 48.8184 0)
+			(show_name no)
+			(do_not_autoplace no)
 			(effects
 				(font
@@
 		(property "Sheetfile" "analogInDivider.kicad_sch"
 			(at 121.92 53.9246 0)
+			(hide yes)
+			(show_name no)
+			(do_not_autoplace no)
 			(effects
 				(font
@@
 				)
 				(justify left top)
-				(hide yes)
 			)
 		)
@@
 		)
 		(fill
-			(color 0 0 0 0.0000)
+			(color 0 0 0 0)
 		)
 		(property "Sheetname" "V Divider10"
 			(at 121.92 117.3984 0)
+			(show_name no)
+			(do_not_autoplace no)
 			(effects
 				(font
@@
 		(property "Sheetfile" "analogInDivider.kicad_sch"
 			(at 121.92 122.5046 0)
+			(hide yes)
+			(show_name no)
+			(do_not_autoplace no)
 			(effects
 				(font
@@
 				)
 				(justify left top)
-				(hide yes)
 			)
 		)
@@
 		)
 		(fill
-			(color 0 0 0 0.0000)
+			(color 0 0 0 0)
 		)
 		(property "Sheetname" "V Divider7"
 			(at 121.92 94.5384 0)
+			(show_name no)
+			(do_not_autoplace no)
 			(effects
 				(font
@@
 		(property "Sheetfile" "analogInDivider.kicad_sch"
 			(at 121.92 99.6446 0)
+			(hide yes)
+			(show_name no)
+			(do_not_autoplace no)
 			(effects
 				(font
@@
 				)
 				(justify left top)
-				(hide yes)
 			)
 		)
@@
 		)
 		(fill
-			(color 0 0 0 0.0000)
+			(color 0 0 0 0)
 		)
 		(property "Sheetname" "V Divider6"
 			(at 121.92 86.9184 0)
+			(show_name no)
+			(do_not_autoplace no)
 			(effects
 				(font
@@
 		(property "Sheetfile" "analogInDivider.kicad_sch"
 			(at 121.92 92.0246 0)
+			(hide yes)
+			(show_name no)
+			(do_not_autoplace no)
 			(effects
 				(font
@@
 				)
 				(justify left top)
-				(hide yes)
 			)
 		)
@@
 		)
 		(fill
-			(color 0 0 0 0.0000)
+			(color 0 0 0 0)
 		)
 		(property "Sheetname" "V Divider2"
 			(at 121.92 56.4384 0)
+			(show_name no)
+			(do_not_autoplace no)
 			(effects
 				(font
@@
 		(property "Sheetfile" "analogInDivider.kicad_sch"
 			(at 121.92 61.5446 0)
+			(hide yes)
+			(show_name no)
+			(do_not_autoplace no)
 			(effects
 				(font
@@
 				)
 				(justify left top)
-				(hide yes)
 			)
 		)
@@
 				(path "/6f45ac2a-5758-484d-9640-5d55da88e919/d6b5e708-7140-4f02-bc93-f8e164db9146"
 					(page "21")
+				)
+			)
+		)
+	)
+	(sheet
+		(at 121.92 125.73)
+		(size 22.86 3.81)
+		(exclude_from_sim no)
+		(in_bom yes)
+		(on_board yes)
+		(dnp no)
+		(fields_autoplaced yes)
+		(stroke
+			(width 0.1524)
+			(type solid)
+		)
+		(fill
+			(color 0 0 0 0)
+		)
+		(property "Sheetname" "V Divider11"
+			(at 121.92 125.0184 0)
+			(show_name no)
+			(do_not_autoplace no)
+			(effects
+				(font
+					(size 1.27 1.27)
+				)
+				(justify left bottom)
+			)
+		)
+		(property "Sheetfile" "analogInDivider.kicad_sch"
+			(at 121.92 130.1246 0)
+			(hide yes)
+			(show_name no)
+			(do_not_autoplace no)
+			(effects
+				(font
+					(size 1.27 1.27)
+				)
+				(justify left top)
+			)
+		)
+		(pin "U_IN" input
+			(at 144.78 127 0)
+			(effects
+				(font
+					(size 1.27 1.27)
+				)
+				(justify right)
+			)
+		)
+		(pin "U_OUT" output
+			(at 121.92 127 180)
+			(effects
+				(font
+					(size 1.27 1.27)
+				)
+				(justify left)
+			)
+		)
+		(instances
+			(project "IOcan"
+				(path "/6f45ac2a-5758-484d-9640-5d55da88e919/d6b5e708-7140-4f02-bc93-f8e164db9146"
+					(page "30")
 				)
 			)
@@
 		)
 		(fill
-			(color 0 0 0 0.0000)
+			(color 0 0 0 0)
 		)
 		(property "Sheetname" "V Divider8"
 			(at 121.92 102.1584 0)
+			(show_name no)
+			(do_not_autoplace no)
 			(effects
 				(font
@@
 		(property "Sheetfile" "analogInDivider.kicad_sch"
 			(at 121.92 107.2646 0)
+			(hide yes)
+			(show_name no)
+			(do_not_autoplace no)
 			(effects
 				(font
@@
 				)
 				(justify left top)
-				(hide yes)
 			)
 		)
@@
 		)
 		(fill
-			(color 0 0 0 0.0000)
+			(color 0 0 0 0)
 		)
 		(property "Sheetname" "V Divider4"
 			(at 121.92 71.6784 0)
+			(show_name no)
+			(do_not_autoplace no)
 			(effects
 				(font
@@
 		(property "Sheetfile" "analogInDivider.kicad_sch"
 			(at 121.92 76.7846 0)
+			(hide yes)
+			(show_name no)
+			(do_not_autoplace no)
 			(effects
 				(font
@@
 				)
 				(justify left top)
-				(hide yes)
 			)
 		)
@@
 		)
 		(fill
-			(color 0 0 0 0.0000)
+			(color 0 0 0 0)
 		)
 		(property "Sheetname" "V Divider9"
 			(at 121.92 109.7784 0)
+			(show_name no)
+			(do_not_autoplace no)
 			(effects
 				(font
@@
 		(property "Sheetfile" "analogInDivider.kicad_sch"
 			(at 121.92 114.8846 0)
+			(hide yes)
+			(show_name no)
+			(do_not_autoplace no)
 			(effects
 				(font
@@
 				)
 				(justify left top)
-				(hide yes)
-			)
-		)
+			)
+		)

Commit message: Checked pinouts
Other:
- note added: "Checked ok"
Changed lines of the file:
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@@
 	(generator_version "10.0")
 	(paper "A4")
+	(text "Checked ok"
+		(exclude_from_sim no)
+		(at 196.596 172.974 0)
+		(effects
+			(font
+				(size 1.27 1.27)
+			)
+		)
+	)
 	(wire
 		(pts
