File: analogInDivider.kicad_sch (KiCad schematic)
At the start: 3 parts

Commit message: Checked pinouts
Parts:
- R37: value 10k -> 36k
Other:
- note added: "Checked ok"
Changed lines of the file:
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@@
 	(generator_version "10.0")
 	(paper "A4")
+	(text "Checked ok"
+		(exclude_from_sim no)
+		(at 189.992 172.974 0)
+		(effects
+			(font
+				(size 1.27 1.27)
+			)
+		)
+	)
 	(junction
 		(at 144.78 88.9)
@@
 			)
 		)
-		(property "Value" "10k"
+		(property "Value" "36k"
 			(at 141.478 75.692 0)
 			(hide yes)
