File: buck_max25231.kicad_sch (KiCad schematic)
At the start: 12 parts, among them IC10 MAX25231ATCB_V+T

Commit message: Checked pinouts
Parts:
- added C95: 4.7u/6.3V, Capacitor_SMD:C_0603_1608Metric, symbol Device:C
- C73, C74, C75: value 100n/6.3V -> 4.7u/6.3V
- R69: value 33k -> 10k
Connections:
- net Uout: now also C95.1
- net VSS: now also C95.2
Other:
- note added: "schematic ok, Component values to check"
- moved on the sheet: C73, C74, C75, C76
