File: canbus.kicad_sch (KiCad schematic)
At the start: 10 parts

Commit message: Checked pinouts
Parts:
- C? (x2): value 100n -> 100n/6.3V
Other:
- note added: "Checked ok"
Changed lines of the file:
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@@
 	(generator_version "10.0")
 	(paper "A4")
+	(text "Checked ok"
+		(exclude_from_sim no)
+		(at 197.612 170.942 0)
+		(effects
+			(font
+				(size 1.27 1.27)
+			)
+		)
+	)
 	(junction
 		(at 107.95 72.39)
@@
 			)
 		)
-		(property "Value" "100n"
+		(property "Value" "100n/6.3V"
 			(at 156.21 64.7699 0)
 			(show_name no)
@@
 			)
 		)
-		(property "Value" "100n"
+		(property "Value" "100n/6.3V"
 			(at 85.09 80.0099 0)
 			(show_name no)
