File: digitalOutputs.kicad_sch (KiCad schematic)
At the start: 10 parts, among them IC8 TLE94106ESXUMA1, U4 SN74AHCT1G126DBVR

Commit message: Checked pinouts
Parts:
- R35: now not fitted
Changed lines of the file:
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@@
 		(on_board yes)
 		(in_pos_files yes)
-		(dnp no)
+		(dnp yes)
 		(property "Reference" "R35"
 			(at 59.944 97.028 90)
