File: interface.kicad_sch (KiCad schematic)
At the start: 1 part

Commit message: Checked pinouts
Other:
- note added: "Pinout checked ok"
Changed lines of the file:
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@@
 	(generator_version "10.0")
 	(paper "A4")
+	(text "Pinout checked ok\n"
+		(exclude_from_sim no)
+		(at 198.374 170.688 0)
+		(effects
+			(font
+				(size 1.27 1.27)
+			)
+		)
+	)
 	(junction
 		(at 165.1 86.36)
