File: kl30bSupply.kicad_sch (KiCad schematic)
At the start: 17 parts, among them IC7 BTG7003A1EPWXUMA1, U2 SN74AHCT1G126DBVR, U3 SN74AHCT1G126DBVR

Commit message: Checked pinouts
Parts:
- R30: value 10k -> 1k2
- R31, R32: now not fitted
Changed lines of the file:
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@@
 			)
 		)
-		(property "Value" "10k"
+		(property "Value" "1k2"
 			(at 168.402 127.508 0)
 			(hide yes)
@@
 		(on_board yes)
 		(in_pos_files yes)
-		(dnp no)
+		(dnp yes)
 		(property "Reference" "R32"
 			(at 103.124 100.838 90)
@@
 		(on_board yes)
 		(in_pos_files yes)
-		(dnp no)
+		(dnp yes)
 		(property "Reference" "R31"
 			(at 138.176 100.838 90)
