File: mcu.emmc.kicad_sch (KiCad schematic)
At the start: 12 parts, among them IC6 IS21ES08GA-JCLI-TR

Commit message: Checked pinouts
Parts:
- C38, C40, C42: value 100n -> 100n/6.3V
Changed lines of the file:
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@@
 			)
 		)
-		(property "Value" "100n"
+		(property "Value" "100n/6.3V"
 			(at 41.91 189.2299 0)
 			(show_name no)
@@
 			)
 		)
-		(property "Value" "100n"
+		(property "Value" "100n/6.3V"
 			(at 41.91 170.1799 0)
 			(show_name no)
@@
 			)
 		)
-		(property "Value" "100n"
+		(property "Value" "100n/6.3V"
 			(at 48.26 114.2999 0)
 			(show_name no)
