File: mcu.qspi.mem.kicad_sch (KiCad schematic)
At the start: 2 parts, among them IC4 SST26VF064BT-104I_SM

Commit message: Checked pinouts
Parts:
- C43: value 100n -> 100n/6.3V
Changed lines of the file:
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@@
 			)
 		)
-		(property "Value" "100n"
+		(property "Value" "100n/6.3V"
 			(at 161.29 93.9799 0)
 			(show_name no)
