File: spiToCan.kicad_sch (KiCad schematic)
At the start: 5 parts, among them IC5 MCP2518FDT-H_SL, Y1 12MHz

Commit message: Checked pinouts
Parts:
- C10, C11: value ~p -> 6pF
- C12: value 100n -> 100n/6.3V
- Y1: value 12MHz -> 40MHz
Other:
- note added: "Checked ok"
Changed lines of the file:
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@@
 	(generator_version "10.0")
 	(paper "A4")
+	(text "Checked ok"
+		(exclude_from_sim no)
+		(at 195.326 173.482 0)
+		(effects
+			(font
+				(size 1.27 1.27)
+			)
+		)
+	)
 	(junction
 		(at 104.14 116.84)
@@
 			)
 		)
-		(property "Value" "100n"
+		(property "Value" "100n/6.3V"
 			(at 190.5 114.2999 0)
 			(show_name no)
@@
 			)
 		)
-		(property "Value" "~p"
+		(property "Value" "6pF"
 			(at 121.92 128.2699 0)
 			(show_name no)
@@
 			)
 		)
-		(property "Value" "~p"
+		(property "Value" "6pF"
 			(at 107.95 128.2699 0)
 			(show_name no)
@@
 			)
 		)
-		(property "Value" "12MHz"
+		(property "Value" "40MHz"
 			(at 111.76 110.49 0)
 			(show_name no)
